Commit message: -updated link and joint names in URDF to be more accurate for our arm
-started implementing end effector rotation matrix

File: src/arm/src/examples/arm_urdf.urdf (robot description, URDF)
Before this commit: robot robot_arm, 7 links, 6 joints
Links:
- removed link arm1
- removed link arm2
- removed link base_link
- removed link base_rot
- removed link camera
- removed link tilt
- removed link top
- added link EFL; visual cylinder length=0.1 radius=0.0175
- added link TSL; visual box size=0.05 0.05 0.053
- added link base; visual cylinder length=0.050 radius=0.089
- added link end_effector; visual box size=0.02 0.02 0.1
- added link forearm; visual box size=0.09 0.03 0.045
- added link hand; visual cylinder length=0.1 radius=0.02
- added link upper_arm; visual cylinder length=0.5 radius=0.022
Joints:
- removed joint base_joint
- removed joint elbow_joint
- removed joint rot2_joint
- removed joint rot_joint
- removed joint shoulder_joint
- removed joint tilt_joint
- added joint elbow: type revolute, parent upper_arm, child EFL, origin xyz=0 0 0.5 rpy=0 0 0, axis 1 0 0, limit lower=-2.8 upper=2.8
- added joint forearm_rotation: type revolute, parent EFL, child forearm, origin xyz=0 0 0.35 rpy=0 0 0, axis 0 0 -1, limit lower=-1.57 upper=2.8
- added joint hand_rotation: type revolute, parent hand, child end_effector, origin xyz=0 0 0.045 rpy=0 0 0, axis 0 0 1
- added joint shoulder: type revolute, parent TSL, child upper_arm, origin xyz=0 0 0.027 rpy=0 0 0, axis 1 0 0, limit lower=-0.9 upper=0.9
- added joint turntable: type revolute, parent base, child TSL, origin xyz=0 0 0.072 rpy=0 0 0, axis 0 0 -1
- added joint wrist: type revolute, parent forearm, child hand, origin xyz=0 0 0.05 rpy=0 0 0, axis -1 0 0, limit lower=-2.5 upper=2.5

Commit message: Updated hand rotation matrix and some joint limits

File: src/arm/src/examples/arm_urdf.urdf (robot description, URDF)
Before this commit: robot robot_arm, 7 links, 6 joints
Links:
- removed link base
- added link base_link; visual cylinder length=0.050 radius=0.089
Joints:
- joint turntable: parent base -> base_link
- joint wrist: limit lower=-2.5 upper=2.5 -> lower=-4 upper=4

Commit message: updated some joint limits

File: src/arm/src/examples/arm_urdf.urdf (robot description, URDF)
Before this commit: robot robot_arm, 7 links, 6 joints
Links:
- link end_effector: geometry visual box size=0.02 0.02 0.02
- link hand: geometry visual cylinder length=0.02 radius=0.02
- link upper_arm: geometry visual cylinder length=0.28 radius=0.022
Joints:
- joint elbow: limit lower=-2.8 upper=2.8 -> lower=-3.14 upper=3.14
- joint forearm_rotation: limit lower=-1.57 upper=2.8 -> lower=-6 upper=6
- joint hand_rotation: limit (none) -> lower=-6 upper=6
- joint shoulder: limit lower=-0.9 upper=0.9 -> lower=-2 upper=2
- joint turntable: limit (none) -> lower=-10 upper=10
- joint wrist: limit lower=-4 upper=4 -> lower=-3 upper=3

Commit message: Update dimensions

File: src/arm/src/examples/arm_urdf.urdf (robot description, URDF)
Before this commit: robot robot_arm, 7 links, 6 joints
Links:
- link EFL: geometry visual box size=.085 .16 .115
- link TSL: geometry visual cylinder length=.0175 radius=.06
- link base_link: geometry visual box size=.20 .20 .05
- link forearm: geometry visual box size=0.07 0.07 0.38
- link hand: geometry visual cylinder length=0.42 radius=0.04
- link upper_arm: geometry visual box size=.11 .09 .51
Joints:
- joint elbow: origin xyz=0 0 0.5 rpy=0 0 0 -> xyz=0 0.0 0.51 rpy=0 0 0
- joint forearm_rotation: origin xyz=0 0 0.35 rpy=0 0 0 -> xyz=0 -0.1 0 rpy=0 0 0
- joint hand_rotation: origin xyz=0 0 0.045 rpy=0 0 0 -> xyz=0 0 0.048 rpy=0 0 0
- joint shoulder: origin xyz=0 0 0.027 rpy=0 0 0 -> xyz=0 0.06 0.075 rpy=0 0 0
- joint turntable: origin xyz=0 0 0.072 rpy=0 0 0 -> xyz=0 .0 .05 rpy=0 0 0
- joint wrist: axis -1 0 0 -> 1 0 0; origin xyz=0 0 0.05 rpy=0 0 0 -> xyz=0 0 0.48 rpy=0 0 0

Commit message: -Added support for new URDF -Added proper start position -fixed incorrect orientations of forarm and wrist rotation -fixed bounds in URDF file

File: src/arm/src/examples/arm_urdf.urdf (robot description, URDF)
Before this commit: robot robot_arm, 7 links, 6 joints
Joints:
- joint elbow: limit lower=-3.14 upper=3.14 -> lower=-3.14 upper=1
- joint forearm_rotation: limit lower=-6 upper=6 -> lower=-3.14 upper=3.14
- joint shoulder: limit lower=-2 upper=2 -> lower=-1.5 upper=1.5
- joint turntable: limit lower=-10 upper=10 -> lower=-1.5 upper=1.5
- joint wrist: limit lower=-3 upper=3 -> lower=-2 upper=2
