Commit message: Added basic roll pitch & yaw
Added the option to include roll pitch and yaw, as well as full rotation. Arm should work with y values too now

File: src/arm/resource/arm.urdf (robot description, URDF)
Before this commit: robot viator, 8 links, 7 joints
Joints:
- joint elbow_joint: limit lower=-3.14 upper=0.1 -> lower=-3.14 upper=0.1 effort=1 velocity=1
- joint shoulder_joint: limit lower=0 upper=1.57 -> lower=0 upper=1.57 effort=1 velocity=1
- joint spinny_joint: limit lower=-3.14 upper=3.14 -> lower=-3.14 upper=3.14 effort=1 velocity=1
- joint wrist_x_joint: limit lower=-3.14 upper=3.14 -> lower=-3.14 upper=3.14 effort=1 velocity=1
- joint wrist_y_joint: limit lower=-1 upper=1 -> lower=-1 upper=1 effort=1 velocity=1

Commit message: got rid of wrist in old urdf

File: src/arm/resource/arm.urdf (robot description, URDF)
Before this commit: robot viator, 8 links, 7 joints
Links:
- removed link hand
- removed link wristbone
Joints:
- removed joint wrist_x_joint
- removed joint wrist_y_joint

Commit message: minor changes to dimensions of urdf

File: src/arm/resource/arm.urdf (robot description, URDF)
Before this commit: robot viator, 6 links, 5 joints
Links:
- link forearm: geometry visual box size=0.330 0.06 0.05
- link shoulder2: geometry visual box size=0.381 0.06 0.05

Commit message: [autonomous][arm-typing] Implements logic to move arm and transform key location to arm Pose

File: src/arm/resource/arm.urdf (robot description, URDF)
Before this commit: robot viator, 6 links, 5 joints
Links:
- added link arm_camera_link
Joints:
- added joint arm_camera_joint: type fixed, parent forearm, child arm_camera_link, origin xyz=-0.15 0 -0.03 rpy=0 0 0

Commit message: [autonomous][arm-typing] Updates urdf file and uses moveit2 for arm movement control.

File: src/arm/resource/arm.urdf (robot description, URDF)
Before this commit: robot viator, 7 links, 6 joints
Links:
- removed link arm_camera_link
- removed link base_box
- removed link elbow
- removed link shoulder1
- removed link shoulder2
- added link bicep_actuator, mass 0.622108; collision mesh filename=${mesh_path}/0_4m_shaft.stl; collision mesh filename=${mesh_path}/200mm_linear_actuator_base.stl
- added link elbow_linkage, mass 0.0164299; collision mesh filename=${mesh_path}/actuator_linkage.stl; collision mesh filename=${mesh_path}/actuator_linkage.stl
- added link gripper_assembly, mass 0.942224; collision mesh filename=${mesh_path}/1911_0025_0836_assembly.stl; collision mesh filename=${mesh_path}/1911_0025_0836_assembly__2.stl
- added link joint, mass 0.118383; collision mesh filename=${mesh_path}/deleteface2.stl; collision mesh filename=${mesh_path}/part_1__26.stl
- added link shoulder_assembly, mass 2.78799; collision mesh filename=${mesh_path}/1mt_054_006.stl; collision mesh filename=${mesh_path}/1mt_054_006__2.stl
- link base_link: mass None -> 1e-09; geometry 
- link forearm: mass None -> 1.24353; geometry collision mesh filename=${mesh_path}/0_3m_shaft.stl; collision mesh filename=${mesh_path}/extrude_thin1.stl
Joints:
- removed joint arm_camera_joint
- removed joint elbow_fixed
- removed joint elbow_joint
- removed joint shoulder_fixed
- removed joint shoulder_joint
- removed joint spinny_joint
- added joint base_link_to_elbow_linkage: type fixed, parent base_link, child elbow_linkage, origin xyz=0 0 0 rpy=0 -0 0, axis 0 0 1, limit effort=10 velocity=10
- added joint base_link_to_shoulder_assembly: type fixed, parent base_link, child shoulder_assembly, origin xyz=0 0 0 rpy=0 -0 0, axis 0 0 1, limit effort=10 velocity=10
- added joint elbow_1: type revolute, parent bicep_actuator, child forearm, origin xyz=0.219114 -0.313521 -0.018175 rpy=-0 -0 2.18077, axis 0 0 1, limit lower=-3.141592653589793 upper=3.141592653589793 effort=10 velocity=10
- added joint shoulder_1: type revolute, parent shoulder_assembly, child bicep_actuator, origin xyz=-0.025675 0.000500014 0.09335 rpy=1.5708 -1.179 -1.5708, axis 0 0 1, limit lower=-3.141592653589793 upper=3.141592653589793 effort=10 velocity=10
- added joint wrist_1: type revolute, parent forearm, child joint, origin xyz=-0.317969 -0.143256 0.0265 rpy=-0 0 -2.7183, axis 0 0 1, limit lower=-3.141592653589793 upper=3.141592653589793 effort=10 velocity=10
- added joint wrist_2: type revolute, parent joint, child gripper_assembly, origin xyz=-0.00623455 -0.00468726 -0.034 rpy=-1.5708 1.16626 2.21546, axis 0 0 1, limit lower=-3.141592653589793 upper=3.141592653589793 effort=10 velocity=10
